Commit message: fixes

File: pendulum.urdf (robot description, URDF)
Before this commit: robot pendulum, 4 links, 3 joints
Joints:
- joint world_to_base: origin xyz=0 0 1 rpy=0 3.1415 0 -> xyz=0 0 1 rpy=0 3.14159265358979323846 0

Commit message: 6-axis robot

File: pendulum.urdf (robot description, URDF)
Before this commit: robot pendulum, 4 links, 3 joints
Links:
- added link link_2, mass 5; visual cylinder length=0.8 radius=0.05
- added link link_3
- added link link_4; visual cylinder length=0.4 radius=0.05
- added link link_5; visual cylinder length=0.2 radius=0.05
- added link link_6
- link base: geometry visual cylinder length=0.2 radius=0.3
- link link_1: mass 0 -> None; geometry visual cylinder length=0.4 radius=0.1
- link link_eef: mass 1 -> 0; geometry visual box size=0.1 0.1 0.1
Joints:
- added joint joint_2: type revolute, parent link_1, child link_2, origin xyz=0 0 0.4 rpy=0 -1.57 0, axis 0 1 0, limit lower=-3.15 upper=3.15
- added joint joint_3: type revolute, parent link_2, child link_3, origin xyz=0 0 0.8 rpy=0 0 0, axis 0 1 0, limit lower=-3.15 upper=3.15
- added joint joint_4: type revolute, parent link_3, child link_4, origin xyz=0 0 0 rpy=0 0 0, axis 0 0 1, limit lower=-3.15 upper=3.15
- added joint joint_5: type revolute, parent link_4, child link_5, origin xyz=0 0 0.4 rpy=0 0 0, axis 0 1 0, limit lower=-3.15 upper=3.15
- added joint joint_6: type revolute, parent link_5, child link_6, origin xyz=0 0 0 rpy=0 0 0, axis 0 0 1, limit lower=-3.15 upper=3.15
- joint joint_1: axis 0 1 0 -> 1 0 0; limit effort=0 velocity=0 -> lower=-3.15 upper=3.15; origin (none) -> xyz=0.0 0 0.2 rpy=0 1.57 0
- joint joint_eef: origin xyz=0 0 0.8 rpy=0 0 0 -> xyz=0 0 0.2 rpy=0 0 0; parent link_1 -> link_6
- joint world_to_base: origin xyz=0 0 1 rpy=0 3.1415 0 -> xyz=0 0 0.1 rpy=0 0 0
